File: 40pin_PICMCU.sch (KiCad schematic (older format))
At the start: 19 parts, among them P1 CONN_10, P2 CONN_10, P3 CONN_10, P4 CONN_10, P5 CONN_7, P6 ICSP, P7 CONN_01X01, SW1 rst, X1 20Mhz

Commit message: Updated Designs
Parts:
- removed P5: CONN_7, symbol CONN_7
- added C5, C6: 0.1uF, symbol C
- added CON1: USB-MICRO-B, symbol USB-MICRO-B
- added JP1: JUMPER, symbol JUMPER
- added P10, P5, P8, P9: CONN_01X01, symbol CONN_01X01
- added R4: R, symbol R
- added U1: CP2102, symbol CP2102
Connections:
- net +5V: now also C3.1, C4.1, U***1.28 (VDD), U***1.7 (VDD), C5.1, CON1.1 (VBUS), U1.7 (REGIN), U1.8 (VBUS)
- net GND: now also C5.2, C6.1, CON1.4 (ID), CON1.5 (GND), U1.3 (GND)
- net MCLR: now also JP1.2
- net RX: now also R4.1
- net TX: now also U1.25 (RXD)
- new net: CON1.2 (D-), U1.5 (D-)
- new net: CON1.3 (D+), U1.4 (D+)
- new net: R4.2, U1.26 (TXD)
- new net: JP1.1, U1.28 (DTR)
- new net: C6.2, U1.6 (VDD)
- no-connect marks 10 -> 34
Other:
- moved on the sheet: P7

Commit message: Updated
Parts:
- added R5: 470r, symbol R
- R4: value R -> 470r
Connections:
- net GND: no longer CON1.4 (ID)
- net TX: now also R5.1; no longer U1.25 (RXD)
- net SCL: now reaches P1.5 (P5), U***1.37 (RC3/SCK/SCL)
- net SCL: now also P4.1 (P1)
- net SDA: now reaches P1.4 (P4), U***1.42 (RC4/SDI/SDA)
- net SDA: now also P4.2 (P2)
- new net: R5.2, U1.25 (RXD)
- no-connect marks 34 -> 33
Other:
- note added: "Logo"
- note added: "Mounting Holes"
Changed lines of the file:
@@
 	1    0    0    -1
 $EndComp
-NoConn ~ 6300 3450
-NoConn ~ 6300 3350
 NoConn ~ 5950 3050
 NoConn ~ 5950 3150
@@
 Wire Wire Line
 	2050 6450 2550 6450
-Wire Wire Line
-	2550 6550 2050 6550
-Wire Wire Line
-	2050 6550 2050 6650
 $Comp
 L GND #PWR3
@@
 	-1   0    0    -1
 $EndComp
-Wire Wire Line
-	2300 6600 2300 6550
-Connection ~ 2300 6550
 $Comp
 L C C6
@@
 NoConn ~ 4900 6150
 NoConn ~ 4900 6550
-Text Label 4900 6250 0    60   ~ 0
+Text Label 5500 6250 0    60   ~ 0
 TX
 $Comp
@@
 P 5300 6350
 F 0 "R4" V 5380 6350 50  0000 C CNN
-F 1 "R" V 5307 6351 50  0000 C CNN
+F 1 "470r" V 5307 6351 50  0000 C CNN
 F 2 "" V 5230 6350 30  0000 C CNN
 F 3 "" H 5300 6350 30  0000 C CNN
@@
 NoConn ~ 7300 3800
 NoConn ~ 7300 4400
+NoConn ~ 2050 6550
+Wire Wire Line
+	2050 6650 2200 6650
+Wire Wire Line
+	2200 6650 2200 6550
+Wire Wire Line
+	2200 6550 2550 6550
+Wire Wire Line
+	2300 6600 2300 6550
+Connection ~ 2300 6550
+Text Notes 7700 3250 0    60   ~ 0
+Logo
+Text Notes 7600 3550 0    60   ~ 0
+Mounting Holes
+Text Label 3250 4000 0    60   ~ 0
+SCL
+Text Label 3250 4100 0    60   ~ 0
+SDA
+Text Label 6300 3350 2    60   ~ 0
+SCL
+Text Label 6300 3450 2    60   ~ 0
+SDA
+$Comp
+L R R5
+U 1 1 579C5043
+P 5250 6250
+F 0 "R5" V 5150 6250 50  0000 C CNN
+F 1 "470r" V 5257 6251 50  0000 C CNN
+F 2 "" V 5180 6250 30  0000 C CNN
+F 3 "" H 5250 6250 30  0000 C CNN
+	1    5250 6250
+	0    1    1    0
+$EndComp
+Wire Wire Line
+	4900 6250 5000 6250
 $EndSCHEMATC
