File: 40pin_PICMCU.kicad_pcb (KiCad board)
At the start: 2 copper layers, 25.4 x 52.1 mm, 19 parts, among them P1 CONN_10, P2 CONN_10, P3 CONN_10, P4 CONN_10, P5 CONN_7, P6 ICSP, P7 CONN_01X01, SW1 rst, X1 20Mhz

Commit message: Updated Designs
Parts:
- added C5: 0.1uF, Capacitors_SMD:C_0603_HandSoldering, B.Cu at (144.8, 103.6)
- added C6: 0.1uF, Capacitors_SMD:C_0603_HandSoldering, B.Cu at (134.9, 100.6)
- added CON1: USB-MICRO-B, EE:USB_Micro-B_SMD_NEW, F.Cu at (139.7, 90.8)
- added JP1: JUMPER, Pin_Headers:Pin_Header_Straight_1x02, F.Cu at (146.1, 141.0)
- added P10: CONN_01X01, Connect:1pin, F.Cu at (128.9, 87.0)
- added P8: CONN_01X01, Connect:1pin, F.Cu at (128.9, 144.8)
- added P9: CONN_01X01, Connect:1pin, F.Cu at (150.5, 144.8)
- added R4: R, Resistors_SMD:R_0603_HandSoldering, B.Cu at (133.9, 97.3)
- added U1: CP2102, EE:cp2102_xl2, B.Cu at (139.7, 99.8)
- P5: value CONN_7 -> CONN_01X01; footprint Pin_Headers:Pin_Header_Straight_1x07 -> Connect:1pin
- moved P5 52.2 mm to (150.5, 87.0), turned to 0 degrees
- moved P6 51.9 mm to (142.9, 141.0)
- moved SW1 6.60 mm to (139.7, 134.6)
- moved C1 6.23 mm to (146.1, 127.6)
- moved C2 6.23 mm to (133.3, 127.6)
- moved X1 6.22 mm to (137.2, 127.6)
- moved U***1 4.45 mm to (139.7, 114.9)
- moved C4 2.92 mm to (136.5, 113.7)
- moved C3 2.87 mm to (142.9, 113.0)
- moved R1 2.16 mm to (139.7, 132.7)
- moved P7 1.05 mm to (139.4, 99.1)
Connections:
- C3 pad 1: Net-(C3-Pad1) -> /+5V
- C4 pad 1: Net-(C3-Pad1) -> /+5V
- P5 pad 1: GND -> Net-(P5-Pad1)
- U***1 pad 28: Net-(C3-Pad1) -> /+5V
- U***1 pad 7: Net-(C3-Pad1) -> /+5V
Other:
- board size 25.4 x 52.1 mm -> 25.4 x 61.6 mm
- board text added: "."
- board text added: "16F877A 16F887 18F4520 18F458"
- board text added: "BOOT"
- board text added: "JMP"
- board text added: "PC5"
- board text added: "PC6"
- board text added: "PC7"
- board text added: "PD0"
- board text added: "PD1"
- board text added: "PD2"
- board text removed: "0"
- board text removed: "1"
- board text removed: "2"
- board text removed: "5"
- board text removed: "6"
- board text removed: "7"
- board text removed: "AUX"
- board text removed: "DTR"

Commit message: proposed a little change in layout
Other:
- board size 25.4 x 61.6 mm -> 25.4 x 62.9 mm
Changed lines of the file:
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@@
     (links 81)
     (no_connects 81)
-    (area 112.015001 60.650001 155.657334 148.603)
+    (area 126.949999 84.404999 152.450001 147.370001)
     (thickness 1.6)
-    (drawings 74)
+    (drawings 88)
     (tracks 0)
     (zones 0)
     (modules 28)
-    (nets 76)
+    (nets 75)
   )
   (page A3)
@@
     (mod_text_size 1 1)
     (mod_text_width 0.15)
-    (pad_size 2.032 2.032)
-    (pad_drill 1.016)
+    (pad_size 3 3)
+    (pad_drill 2)
     (pad_to_mask_clearance 0)
     (aux_axis_origin 0 0)
@@
   (net 70 "Net-(U1-Pad10)")
   (net 71 "Net-(U1-Pad9)")
-  (net 72 "Net-(P5-Pad1)")
-  (net 73 "Net-(P8-Pad1)")
-  (net 74 "Net-(P9-Pad1)")
-  (net 75 "Net-(P10-Pad1)")
+  (net 72 "Net-(P8-Pad1)")
+  (net 73 "Net-(P9-Pad1)")
+  (net 74 "Net-(P10-Pad1)")
   (net_class Default "This is the default net class."
     (clearance 0.254)
@@
       (effects (font (size 1 1) (thickness 0.15)))
     )
-    (pad 1 thru_hole circle (at 0 0) (size 3 3) (drill 2) (layers *.Cu *.Mask F.SilkS)
-      (net 72 "Net-(P5-Pad1)"))
+    (pad "" np_thru_hole circle (at 0 0) (size 3 3) (drill 2) (layers *.Cu *.Mask F.SilkS))
   )
   (module Connect:1pin (layer F.Cu)
@@
     )
     (pad 1 thru_hole circle (at 0 0) (size 3 3) (drill 2) (layers *.Cu *.Mask F.SilkS)
-      (net 75 "Net-(P10-Pad1)"))
+      (net 74 "Net-(P10-Pad1)"))
   )
   (module Connect:1pin (layer F.Cu)
@@
     )
     (pad 1 thru_hole circle (at 0 0) (size 3 3) (drill 2) (layers *.Cu *.Mask F.SilkS)
-      (net 74 "Net-(P9-Pad1)"))
+      (net 73 "Net-(P9-Pad1)"))
   )
   (module Connect:1pin (layer F.Cu)
@@
     )
     (pad 1 thru_hole circle (at 0 0) (size 3 3) (drill 2) (layers *.Cu *.Mask F.SilkS)
-      (net 73 "Net-(P8-Pad1)"))
+      (net 72 "Net-(P8-Pad1)"))
   )
   (module Pin_Headers:Pin_Header_Straight_1x06 (layer F.Cu)
@@
     (pad "" thru_hole rect (at -3.9 4.825 270) (size 2.5 2.2) (drill oval 1.8 0.9) (layers *.Cu *.Mask F.SilkS))
   )
-  (gr_line (start 136.144 85.09) (end 127 85.09) (angle 90) (layer Edge.Cuts) (width 0.1))
-  (gr_line (start 143.256 85.09) (end 152.4 85.09) (angle 90) (layer Edge.Cuts) (width 0.1))
+  (gr_line (start 132.08 84.455) (end 127 84.455) (angle 90) (layer Edge.Cuts) (width 0.1))
+  (gr_line (start 132.715 85.09) (end 132.08 84.455) (angle 90) (layer Edge.Cuts) (width 0.1))
+  (gr_line (start 133.985 85.09) (end 132.715 85.09) (angle 90) (layer Edge.Cuts) (width 0.1))
+  (gr_line (start 136.144 85.09) (end 135.89 85.09) (angle 90) (layer Edge.Cuts) (width 0.1))
+  (gr_line (start 143.51 85.09) (end 143.256 85.09) (angle 90) (layer Edge.Cuts) (width 0.1))
+  (gr_line (start 146.05 85.09) (end 143.51 85.09) (angle 90) (layer Edge.Cuts) (width 0.1))
+  (gr_line (start 134.62 85.09) (end 135.89 85.09) (angle 90) (layer Edge.Cuts) (width 0.1))
+  (gr_line (start 149.225 146.685) (end 149.86 146.685) (angle 90) (layer Edge.Cuts) (width 0.1))
+  (gr_line (start 146.685 85.09) (end 146.05 85.09) (angle 90) (layer Edge.Cuts) (width 0.1))
+  (gr_line (start 147.32 84.455) (end 146.685 85.09) (angle 90) (layer Edge.Cuts) (width 0.1))
+  (gr_line (start 152.4 84.455) (end 147.32 84.455) (angle 90) (layer Edge.Cuts) (width 0.1))
+  (gr_line (start 152.4 85.09) (end 152.4 84.455) (angle 90) (layer Edge.Cuts) (width 0.1))
+  (gr_line (start 133.985 85.09) (end 134.62 85.09) (angle 90) (layer Edge.Cuts) (width 0.1))
+  (gr_line (start 127 85.09) (end 127 84.455) (angle 90) (layer Edge.Cuts) (width 0.1))
+  (gr_line (start 148.59 147.32) (end 149.225 146.685) (angle 90) (layer Edge.Cuts) (width 0.1))
+  (gr_line (start 130.175 147.32) (end 148.59 147.32) (angle 90) (layer Edge.Cuts) (width 0.1))
+  (gr_line (start 129.54 146.685) (end 130.175 147.32) (angle 90) (layer Edge.Cuts) (width 0.1))
   (gr_line (start 143.256 89.916) (end 143.256 85.09) (angle 90) (layer Edge.Cuts) (width 0.1))
   (gr_line (start 136.144 89.916) (end 143.256 89.916) (angle 90) (layer Edge.Cuts) (width 0.1))
@@
   )
   (gr_line (start 127 144.145) (end 127 140.335) (angle 90) (layer Edge.Cuts) (width 0.1))
-  (gr_line (start 149.86 146.685) (end 129.54 146.685) (angle 90) (layer Edge.Cuts) (width 0.1))
   (gr_line (start 152.4 142.875) (end 152.4 144.145) (angle 90) (layer Edge.Cuts) (width 0.1))
   (gr_arc (start 129.54 144.145) (end 129.54 146.685) (angle 90) (layer Edge.Cuts) (width 0.1))

Commit message: Updated
Parts:
- added R5: 470r, Resistors_SMD:R_0603_HandSoldering, F.Cu at (133.6, 103.9)
- C1, C2, C3, C4, C5, C6, R1, R2, R3, U1: moved to F.Cu
- P7: moved to B.Cu
- R4: value R -> 470r; moved to F.Cu
- moved R4 12.2 mm to (144.3, 103.6), turned to 90 degrees
- moved P7 9.91 mm to (139.2, 109.0), turned to 270 degrees
- moved R1 5.62 mm to (144.8, 135.1), turned to 270 degrees
- moved C5 5.36 mm to (144.3, 98.3), turned to 90 degrees
- moved C4 5.21 mm to (131.3, 113.8)
- moved C3 5.21 mm to (148.1, 113.0)
- moved R3 2.55 mm to (133.6, 98.0)
- moved C6 2.55 mm to (135.1, 98.0)
- moved R2 2.29 mm to (145.8, 98.3)
- moved D3 1.80 mm to (133.6, 93.5)
- moved D1 1.78 mm to (145.8, 93.7)
- moved U***1 1.65 mm to (139.7, 113.3)
- moved U1 1.27 mm to (139.7, 98.6)
- moved C1 0.28 mm to (145.8, 127.5), turned to 90 degrees
- moved C2 0.28 mm to (133.6, 127.5), turned to 90 degrees
Connections:
- CON1 pad 4: GND -> Net-(CON1-Pad4)
- P1 pad 4: Net-(P1-Pad4) -> /SDA
- P1 pad 5: Net-(P1-Pad5) -> /SCL
- P4 pad 1: Net-(P4-Pad1) -> /SCL
- P4 pad 2: Net-(P4-Pad2) -> /SDA
- U***1 pad 37: Net-(P1-Pad5) -> /SCL
- U***1 pad 42: Net-(P1-Pad4) -> /SDA
- U1 pad 25: /TX -> Net-(R5-Pad2)
Other:
- outline, holes or cut-outs redrawn
- board text added: "*"
- board text added: "0"
- board text added: "1"
- board text added: "2"
- board text added: "ExploreEmbedded.com"
- board text added: "PWM *"
- board text added: "SCL"
- board text added: "SDA"
- board text removed: "NC"
- board text removed: "PB0"
- board text removed: "PB1"
- board text removed: "PE1"
- board text removed: "PE2"
- board text removed: "PIC"

Commit message: Routing
Parts:
- moved R5 10.3 mm to (143.9, 102.7), turned to 180 degrees
- moved R4 4.06 mm to (144.9, 99.6)
- moved P7 4.00 mm to (140.9, 112.6)
- moved C5 3.72 mm to (146.6, 101.2), turned to 270 degrees
- moved X1 3.18 mm to (137.2, 124.5)
- moved C1 3.05 mm to (145.8, 124.5), turned to 270 degrees
- moved C2 3.05 mm to (133.6, 124.5), turned to 270 degrees
- moved R3 1.84 mm to (132.7, 96.4)
- moved D3 1.75 mm to (132.0, 92.7)
- moved C6 1.73 mm to (134.2, 96.6)
- moved R2 1.39 mm to (146.6, 97.1)
- moved D1 0.76 mm to (146.4, 93.3)
Routing:
- net GND: track 0.00 -> 141.4 mm, vias 0 -> 12
- net /+5V: track 0.00 -> 134.9 mm, vias 0 -> 12
- net /RX: track 0.00 -> 108.5 mm, vias 0 -> 4
- net /TX: track 0.00 -> 101.9 mm, vias 0 -> 5
- net Net-(JP1-Pad1): track 0.00 -> 66.5 mm, vias 0 -> 3
- net /D7/PGD: track 0.00 -> 59.7 mm, vias 0 -> 2
- net /D6/PGC: track 0.00 -> 56.2 mm, vias 0 -> 3
- net /SDA: track 0.00 -> 41.5 mm, vias 0 -> 2
- net /SCL: track 0.00 -> 38.6 mm, vias 0 -> 3
- net Net-(P4-Pad10): track 0.00 -> 29.4 mm
- net Net-(P4-Pad9): track 0.00 -> 29.0 mm
- net Net-(P1-Pad3): track 0.00 -> 27.2 mm, vias 0 -> 1
- net Net-(P4-Pad8): track 0.00 -> 23.5 mm
- net Net-(C1-Pad2): track 0.00 -> 22.5 mm, vias 0 -> 2
- net /MCLR: track 0.00 -> 21.8 mm
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- added copper zone on F.Cu, net /+5V
- added copper zone on B.Cu, net GND
Other:
- net class Default: clearance 0.254 -> 0.1778
- rule trace_clearance: 0.254 -> 0.1778
- rule via_min_drill: 0.508 -> 0.3
- rule via_min_size: 0.889 -> 0.6
